File: attiny2313/kicad/attiny2313-dumbups.kicad_sch (KiCad schematic)
At the start: 12 parts, among them J1 UPS_Interface, J2 AVR ISP, Q1 PN2222A, Q2 PN2222A, U2 MM232R, U3 ATtiny2313V-10P

Commit message: Add status LED to board layout
Parts:
- added D1: LED, Connector_PinHeader_2.54mm:PinHeader_1x02_P2.54mm_Vertical, symbol Device:LED
- added R7: 220, Resistor_THT:R_Axial_DIN0207_L6.3mm_D2.5mm_P10.16mm_Horizontal, symbol Device:R
Connections:
- net at J1.4, J2.6 (Pin_6), Q1.1 (E)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: now also R7.2
- net at U3.4 (PA1/XTAL2): now also D1.1 (K)
- new net: D1.2 (A), R7.1
- no-connect marks 20 -> 19
Changed lines of the file:
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@@
   (junction (at 57.15 87.63) (diameter 0) (color 0 0 0 0)
+  )
+  (junction (at 124.46 143.51) (diameter 0) (color 0 0 0 0)
   )
   (junction (at 27.94 100.33) (diameter 0) (color 0 0 0 0)
@@
   (no_connect (at 30.48 118.11))
   (no_connect (at 30.48 115.57))
-  (no_connect (at 119.38 105.41))
   (no_connect (at 88.9 105.41))
   (no_connect (at 66.04 115.57))
@@
     (stroke (width 0) (type default) (color 0 0 0 0))
   )
+  (wire (pts (xy 119.38 105.41) (xy 124.46 105.41))
+    (stroke (width 0) (type default) (color 0 0 0 0))
+  )
   (wire (pts (xy 87.63 95.25) (xy 87.63 76.2))
     (stroke (width 0) (type default) (color 0 0 0 0))
@@
     (stroke (width 0) (type default) (color 0 0 0 0))
   )
+  (wire (pts (xy 124.46 120.65) (xy 124.46 143.51))
+    (stroke (width 0) (type default) (color 0 0 0 0))
+  )
   (wire (pts (xy 46.99 83.82) (xy 46.99 87.63))
     (stroke (width 0) (type default) (color 0 0 0 0))
@@
     (stroke (width 0) (type default) (color 0 0 0 0))
   )
-  (wire (pts (xy 104.14 143.51) (xy 127 143.51))
+  (wire (pts (xy 104.14 143.51) (xy 124.46 143.51))
     (stroke (width 0) (type default) (color 0 0 0 0))
   )
   (wire (pts (xy 71.12 113.03) (xy 71.12 127))
+    (stroke (width 0) (type default) (color 0 0 0 0))
+  )
+  (wire (pts (xy 124.46 143.51) (xy 127 143.51))
     (stroke (width 0) (type default) (color 0 0 0 0))
   )
@@
     (pin "8")
     (pin "9")
+  )
+  (symbol (lib_id "Device:R") (at 124.46 116.84 0) (unit 1)
+    (in_bom yes) (on_board yes) (fields_autoplaced)
+    (property "Reference" "R7" (id 0) (at 127 115.5699 0)
+      (effects (font (size 1.27 1.27)) (justify left))
+    )
+    (property "Value" "220" (id 1) (at 127 118.1099 0)
+      (effects (font (size 1.27 1.27)) (justify left))
+    )
+    (property "Footprint" "Resistor_THT:R_Axial_DIN0207_L6.3mm_D2.5mm_P10.16mm_Horizontal" (id 2) (at 122.682 116.84 90)
+      (effects (font (size 1.27 1.27)) hide)
+    )
+    (property "Datasheet" "~" (id 3) (at 124.46 116.84 0)
+      (effects (font (size 1.27 1.27)) hide)
+    )
+    (pin "1")
+    (pin "2")
   )
   (symbol (lib_id "MCU_Microchip_ATtiny:ATtiny2313V-10P") (at 104.14 115.57 0) (mirror y) (unit 1)
@@
     (pin "2")
   )
+  (symbol (lib_id "Device:LED") (at 124.46 109.22 270) (unit 1)
+    (in_bom yes) (on_board yes) (fields_autoplaced)
+    (property "Reference" "D1" (id 0) (at 127 106.3624 90)
+      (effects (font (size 1.27 1.27)) (justify left))
+    )
+    (property "Value" "LED" (id 1) (at 127 108.9024 90)
+      (effects (font (size 1.27 1.27)) (justify left))
+    )
+    (property "Footprint" "Connector_PinHeader_2.54mm:PinHeader_1x02_P2.54mm_Vertical" (id 2) (at 124.46 109.22 0)
+      (effects (font (size 1.27 1.27)) hide)
+    )
+    (property "Datasheet" "~" (id 3) (at 124.46 109.22 0)
+      (effects (font (size 1.27 1.27)) hide)
+    )
+    (pin "1")
+    (pin "2")
+  )
   (symbol (lib_id "Device:R") (at 67.31 80.01 0) (unit 1)
     (in_bom yes) (on_board yes) (fields_autoplaced)
@@
   )
   (symbol_instances
+    (path "/e0130066-f120-45ab-8ca4-de7cd402c362"
+      (reference "D1") (unit 1) (value "LED") (footprint "Connector_PinHeader_2.54mm:PinHeader_1x02_P2.54mm_Vertical")
+    )
     (path "/835e435e-a7ba-4fe7-976f-486bb471a3b9"
       (reference "J1") (unit 1) (value "UPS_Interface") (footprint "Connector_Dsub:DSUB-9_Male_Horizontal_P2.77x2.84mm_EdgePinOffset7.70mm_Housed_MountingHolesOffset9.12mm")
@@
       (reference "R6") (unit 1) (value "4.7K") (footprint "Resistor_THT:R_Axial_DIN0207_L6.3mm_D2.5mm_P10.16mm_Horizontal")
     )
+    (path "/bcb54b83-0469-4964-9c1b-ce945bea8582"
+      (reference "R7") (unit 1) (value "220") (footprint "Resistor_THT:R_Axial_DIN0207_L6.3mm_D2.5mm_P10.16mm_Horizontal")
+    )
     (path "/0dabb6d5-4d3c-4a7b-8471-b72d4daf00c9"

Commit message: LED correct way around on schematic etc
Connections:
- net at R7.1: now also D1.1 (K); no longer D1.2 (A)
- net at U3.4 (PA1/XTAL2): now also D1.2 (A); no longer D1.1 (K)
Other:
- moved on the sheet: D1
Changed lines of the file:
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@@
     (pin "2")
   )
-  (symbol (lib_id "Device:LED") (at 124.46 109.22 270) (unit 1)
+  (symbol (lib_id "Device:LED") (at 124.46 109.22 270) (mirror x) (unit 1)
     (in_bom yes) (on_board yes) (fields_autoplaced)
-    (property "Reference" "D1" (id 0) (at 127 106.3624 90)
+    (property "Reference" "D1" (id 0) (at 127 109.5374 90)
       (effects (font (size 1.27 1.27)) (justify left))
     )
-    (property "Value" "LED" (id 1) (at 127 108.9024 90)
+    (property "Value" "LED" (id 1) (at 127 112.0774 90)
       (effects (font (size 1.27 1.27)) (justify left))
     )
